Commit message: bin-picking joint limits

File: khi_rs_description/urdf/rs080n_macro.xacro (robot description, xacro)
@@ -32,16 +32,28 @@
     <xacro:property name="j5_length" value="0.165"/>
     <!-- joint limits [rad] -->
-    <xacro:property name="j1_lower_limit" value="${radians(-180)}"/>
+    <!-- <xacro:property name="j1_lower_limit" value="${radians(-180)}"/> -->
+    <!-- <xacro:property name="j1_upper_limit" value="${radians( 180)}"/> -->
+    <!-- <xacro:property name="j2_lower_limit" value="${radians(-105)}"/> -->
+    <!-- <xacro:property name="j2_upper_limit" value="${radians( 140)}"/> -->
+    <!-- <xacro:property name="j3_lower_limit" value="${radians(-155)}"/> -->
+    <!-- <xacro:property name="j3_upper_limit" value="${radians( 135)}"/> -->
+    <!-- <xacro:property name="j4_lower_limit" value="${radians(-360)}"/> -->
+    <!-- <xacro:property name="j4_upper_limit" value="${radians( 360)}"/> -->
+    <!-- <xacro:property name="j5_lower_limit" value="${radians(-145)}"/> -->
+    <!-- <xacro:property name="j5_upper_limit" value="${radians( 145)}"/> -->
+    <!-- <xacro:property name="j6_lower_limit" value="${radians(-360)}"/> -->
+    <!-- <xacro:property name="j6_upper_limit" value="${radians( 360)}"/> -->
+    <xacro:property name="j1_lower_limit" value="${radians(-90)}"/>
     <xacro:property name="j1_upper_limit" value="${radians( 180)}"/>
-    <xacro:property name="j2_lower_limit" value="${radians(-105)}"/>
-    <xacro:property name="j2_upper_limit" value="${radians( 140)}"/>
+    <xacro:property name="j2_lower_limit" value="${radians(-45)}"/>
+    <xacro:property name="j2_upper_limit" value="${radians( 135)}"/>
     <xacro:property name="j3_lower_limit" value="${radians(-155)}"/>
-    <xacro:property name="j3_upper_limit" value="${radians( 135)}"/>
-    <xacro:property name="j4_lower_limit" value="${radians(-360)}"/>
-    <xacro:property name="j4_upper_limit" value="${radians( 360)}"/>
+    <xacro:property name="j3_upper_limit" value="${radians( 0)}"/>
+    <xacro:property name="j4_lower_limit" value="${radians(-180)}"/>
+    <xacro:property name="j4_upper_limit" value="${radians( 180)}"/>
     <xacro:property name="j5_lower_limit" value="${radians(-145)}"/>
     <xacro:property name="j5_upper_limit" value="${radians( 145)}"/>
-    <xacro:property name="j6_lower_limit" value="${radians(-360)}"/>
-    <xacro:property name="j6_upper_limit" value="${radians( 360)}"/>
+    <xacro:property name="j6_lower_limit" value="${radians(-180)}"/>
+    <xacro:property name="j6_upper_limit" value="${radians( 180)}"/>
     <!-- joint velocity limits [rad/s] -->
     <xacro:property name="j1_velocity_limit" value="${radians(180)}"/>
